Commit message: new urdf + world

File: model/iris_depth_camera.urdf (robot description, URDF)
Before this commit: robot iris_depth_camera, 8 links, 7 joints
Links:
- link base_link: mass 1.5 -> None; geometry collision box size=0.47 0.47 0.11; visual mesh filename=package://px4_offboard/meshes/iris.stl scale=1 1 1
- link camera_link: geometry visual mesh filename=package://px4_offboard/meshes/realsense.dae scale=1.0 1.0 1.0
- link iris_depth_camera__iris__rotor_0: geometry collision cylinder length=0.005 radius=0.128; visual mesh filename=package://px4_offboard/meshes/iris_prop_ccw.dae scale=1 1 1
- link iris_depth_camera__iris__rotor_1: geometry collision cylinder length=0.005 radius=0.128; visual mesh filename=package://px4_offboard/meshes/iris_prop_ccw.dae scale=1 1 1
- link iris_depth_camera__iris__rotor_2: geometry collision cylinder length=0.005 radius=0.128; visual mesh filename=package://px4_offboard/meshes/iris_prop_cw.dae scale=1 1 1
- link iris_depth_camera__iris__rotor_3: geometry collision cylinder length=0.005 radius=0.128; visual mesh filename=package://px4_offboard/meshes/iris_prop_cw.dae scale=1 1 1
