Commit message: multivehicle simulation 1st step

File: px4_offboard/urdf/iris_depth_camera_1.urdf (robot description, URDF)
Before this commit: robot iris_depth_camera, 8 links, 7 joints
Links:
- removed link base_link
- removed link camera_link
- removed link iris_depth_camera__iris__/imu_link
- removed link iris_depth_camera__iris__gps0__link
- removed link iris_depth_camera__iris__rotor_0
- removed link iris_depth_camera__iris__rotor_1
- removed link iris_depth_camera__iris__rotor_2
- removed link iris_depth_camera__iris__rotor_3
- added link base_link_1; collision box size=0.47 0.47 0.11; visual mesh filename=package://px4_offboard/meshes/iris.stl scale=1 1 1
- added link camera_link_1, mass 0.01; visual mesh filename=package://px4_offboard/meshes/realsense.dae scale=1.0 1.0 1.0
- added link gps0__link_1, mass 0.015; visual cylinder length=0.002 radius=0.01
- added link imu_link_1, mass 0.015
- added link rotor_0_1, mass 0.005; collision cylinder length=0.005 radius=0.128; visual mesh filename=package://px4_offboard/meshes/iris_prop_ccw.dae scale=1 1 1
- added link rotor_1_1, mass 0.005; collision cylinder length=0.005 radius=0.128; visual mesh filename=package://px4_offboard/meshes/iris_prop_ccw.dae scale=1 1 1
- added link rotor_2_1, mass 0.005; collision cylinder length=0.005 radius=0.128; visual mesh filename=package://px4_offboard/meshes/iris_prop_cw.dae scale=1 1 1
- added link rotor_3_1, mass 0.005; collision cylinder length=0.005 radius=0.128; visual mesh filename=package://px4_offboard/meshes/iris_prop_cw.dae scale=1 1 1
Joints:
- removed joint iris_depth_camera__depth_camera_joint
- removed joint iris_depth_camera__iris__/imu_joint
- removed joint iris_depth_camera__iris__gps0_joint
- removed joint iris_depth_camera__iris__rotor_0_joint
- removed joint iris_depth_camera__iris__rotor_1_joint
- removed joint iris_depth_camera__iris__rotor_2_joint
- removed joint iris_depth_camera__iris__rotor_3_joint
- added joint depth_camera_joint_1: type fixed, parent base_link_1, child camera_link_1, origin xyz=0.1   0    0.035 rpy=-1.5707 0 -1.5707, axis 0 0 0, limit lower=0 upper=0 effort=0 velocity=0
- added joint gps0_joint_1: type fixed, parent base_link_1, child gps0__link_1, origin xyz=0.05 0   0.04 rpy=0 0 0, axis 0 0 0, limit lower=0 upper=0 effort=0 velocity=0
- added joint imu_joint_1: type fixed, parent base_link_1, child imu_link_1, origin xyz=0   0   0.02 rpy=0 0 0, axis 1 0 0, limit lower=0.0 upper=0.0 effort=0.0 velocity=0.0
- added joint rotor_0_joint_1: type revolute, parent base_link_1, child rotor_0_1, origin xyz=0.13  -0.22   0.023 rpy=0 0 0, axis 0 0 1, limit lower=-1e+16 upper=1e+16 effort=0.0 velocity=0.0
- added joint rotor_1_joint_1: type revolute, parent base_link_1, child rotor_1_1, origin xyz=-0.13   0.2    0.023 rpy=0 0 0, axis 0 0 1, limit lower=-1e+16 upper=1e+16 effort=0.0 velocity=0.0
- added joint rotor_2_joint_1: type revolute, parent base_link_1, child rotor_2_1, origin xyz=0.13  0.22  0.023 rpy=0 0 0, axis 0 0 1, limit lower=-1e+16 upper=1e+16 effort=0.0 velocity=0.0
- added joint rotor_3_joint_1: type revolute, parent base_link_1, child rotor_3_1, origin xyz=-0.13  -0.2    0.023 rpy=0 0 0, axis 0 0 1, limit lower=-1e+16 upper=1e+16 effort=0.0 velocity=0.0
